File: int-brain.kicad_sch (KiCad schematic)
At the start: 34 parts, among them J1 PWR, J10 Left, J11 Right, J2 UART0, J3 I2C0, J4 PWR, J5 1MA, J6 1MB, J7 2MA, J8 2MB, J9 MPU9250, U2 ESP32-DevKitC, U4 LM2576HVT-5

Commit message: done placement
Parts:
- added C7: 100uF, Capacitor_THT:C_Radial_D6.3mm_H11.0mm_P2.50mm, symbol Device:C
- added C8: 1mF, Capacitor_THT:C_Radial_D8.0mm_H11.5mm_P3.50mm, symbol Device:C
- added D24: 1N5822, Diode_THT:D_DO-201AD_P15.24mm_Horizontal, symbol Diode:1N5822
- added D25: PWR, LED_SMD:LED_0603_1608Metric_Pad1.05x0.95mm_HandSolder, symbol Device:LED
- added J12: 1MA_ENC, Connector_JST:JST_EH_B4B-EH-A_1x04_P2.50mm_Vertical, symbol Connector:Conn_01x04_Pin
- added J13: 1MB_ENC, Connector_JST:JST_EH_B4B-EH-A_1x04_P2.50mm_Vertical, symbol Connector:Conn_01x04_Pin
- added J14: 2MA_ENC, Connector_JST:JST_EH_B4B-EH-A_1x04_P2.50mm_Vertical, symbol Connector:Conn_01x04_Pin
- added J15: 2MB_ENC, Connector_JST:JST_EH_B4B-EH-A_1x04_P2.50mm_Vertical, symbol Connector:Conn_01x04_Pin
- added J16: USB_A, Connector_USB:USB_A_Molex_67643_Horizontal, symbol Connector:USB_A
- added JP1, JP2, JP3, JP4, JP5: SolderJumper_2_Open, Jumper:SolderJumper-2_P1.3mm_Open_Pad1.0x1.5mm, symbol Jumper:SolderJumper_2_Open
- added L2: 100mH, Inductor_SMD:L_6.3x6.3_H3, symbol Device:L
- added R16, R17: 4.7k, Resistor_SMD:R_1206_3216Metric_Pad1.30x1.75mm_HandSolder, symbol Device:R
- added R18, R19, R20, R21, R22: 10k, Resistor_SMD:R_1206_3216Metric_Pad1.30x1.75mm_HandSolder, symbol Device:R
- added R23: 470R, Resistor_SMD:R_1206_3216Metric_Pad1.30x1.75mm_HandSolder, symbol Device:R
- added SW1: SW_Push, Button_Switch_THT:SW_PUSH_6mm_H5mm, symbol Switch:SW_Push
- added U7: PCA9635, Package_SO:TSSOP-28_4.4x9.7mm_P0.65mm, symbol Driver_LED:PCA9635
- added U8: LM2576HVT-5, Package_TO_SOT_THT:TO-220-5_Horizontal_TabDown, symbol Regulator_Switching:LM2576HVT-5
- R11: value 3.9k -> 10k
Connections:
- net 2MB2_IN is gone; now on net FSYNC: J10.7 (Pin_7), U2.7 (32K_XP/GPIO32/ADC1_CH4)
- net GPIO36 is gone; now on net 2MB_SENSE: J10.3 (Pin_3), U2.3 (SENSOR_VP/GPIO36/ADC1_CH0)
- net +3.3V: now also J12.2 (Pin_2), J13.2 (Pin_2), J14.2 (Pin_2), J15.2 (Pin_2), JP1.1 (A), JP2.1 (A), JP3.1 (A), JP4.1 (A), JP5.1 (A), R16.2, R17.2, U7.1 (A0), U7.28 (VDD)
- net 1MA1_IN: now also U7.13 (LED7); no longer J11.12 (Pin_12), U2.27 (GPIO16)
- net 1MA_EN: now also U7.12 (LED6); no longer J11.11 (Pin_11), U2.28 (GPIO17)
- net 1MA_SENSE: now also J10.6 (Pin_6), U2.6 (VDET_2/GPIO35/ADC1_CH7); no longer J11.16 (Pin_16), U2.23 (MTDO/GPIO15/ADC2_CH3)
- net 1MB1_IN: now also U7.11 (LED5); no longer J11.9 (Pin_9), U2.30 (GPIO18)
- net 1MB_EN: now also U7.10 (LED4); no longer J11.8 (Pin_8), U2.31 (GPIO19)
- net 1MB_SENSE: now also J10.5 (Pin_5), U2.5 (VDET_1/GPIO34/ADC1_CH6); no longer J11.13 (Pin_13), U2.26 (ADC2_CH0/GPIO4)
- net 2MA1_IN: now also U7.15 (LED8); no longer J10.12 (Pin_12), U2.12 (MTMS/GPIO14/ADC2_CH6)
- net 2MA_EN: now also U7.16 (LED9); no longer J10.11 (Pin_11), U2.11 (ADC2_CH7/GPIO27)
- net 2MA_SENSE: now also J10.4 (Pin_4), U2.4 (SENSOR_VN/GPIO39/ADC1_CH3); no longer J10.6 (Pin_6), U2.6 (VDET_2/GPIO35/ADC1_CH7)
- net 2MB1_IN: now also U7.17 (LED10); no longer J10.9 (Pin_9), U2.9 (DAC_1/ADC2_CH8/GPIO25)
- net 2MB_EN: now also U7.18 (LED11); no longer J10.8 (Pin_8), U2.8 (32K_XN/GPIO33/ADC1_CH5)
- net 2MB_SENSE: no longer J10.5 (Pin_5), U2.5 (VDET_1/GPIO34/ADC1_CH6)
- net FSYNC: no longer J10.13 (Pin_13), U2.13 (MTDI/GPIO12/ADC2_CH5)
- net GND: now also C7.2, C8.2, D24.2 (A), D25.1 (K), J12.1 (Pin_1), J13.1 (Pin_1), J14.1 (Pin_1), J15.1 (Pin_1), J16.4 (GND), J16.5 (Shield), R18.1, R19.1, R20.1, R21.1, R22.1, U7.14 (VSS), U7.25 (A6), U8.3 (GND), U8.5 (~{ON}/OFF)
- net INT: now also J10.8 (Pin_8), U2.8 (32K_XN/GPIO33/ADC1_CH5); no longer J10.15 (Pin_15), U2.15 (MTCK/GPIO13/ADC2_CH4)
- net SCL0: now also R16.1, U7.26 (SCL)
- net SDA0: now also R17.1, U7.27 (SDA)
- net VBATT: now also J10.9 (Pin_9), U2.9 (DAC_1/ADC2_CH8/GPIO25); no longer J10.4 (Pin_4), U2.4 (SENSOR_VN/GPIO39/ADC1_CH3)
- net VIN_BUCK: now also SW1.1
- net 1MA2_IN renamed 1MB2_ENC
- net 1MB2_ENC: now also J13.4 (Pin_4)
- net 1MB2_IN renamed GPIO23
- net 2MA2_IN renamed 2MA1_ENC
- net 2MA1_ENC: now also J14.3 (Pin_3)
- net BUCK_OUT renamed BUCK_OUT_1
- net PWR_LED renamed PWR_LED_1
- new net 1MA1_ENC: J11.8 (Pin_8), J12.3 (Pin_3), U2.31 (GPIO19)
- new net 1MA2_ENC: J11.9 (Pin_9), J12.4 (Pin_4), U2.30 (GPIO18)
- new net 1MB1_ENC: J11.11 (Pin_11), J13.3 (Pin_3), U2.28 (GPIO17)
- new net 2MA2_ENC: J10.11 (Pin_11), J14.4 (Pin_4), U2.11 (ADC2_CH7/GPIO27)
- new net 2MB1_ENC: J10.12 (Pin_12), J15.3 (Pin_3), U2.12 (MTMS/GPIO14/ADC2_CH6)
- new net 2MB2_ENC: J10.13 (Pin_13), J15.4 (Pin_4), U2.13 (MTDI/GPIO12/ADC2_CH5)
- new net BUCK_OUT_2: D24.1 (K), L2.1, U8.2 (OUT)
- new net GPIO13: J10.15 (Pin_15), U2.15 (MTCK/GPIO13/ADC2_CH4)
- new net GPIO15: J11.16 (Pin_16), U2.23 (MTDO/GPIO15/ADC2_CH3)
- new net GPIO16: J11.12 (Pin_12), U2.27 (GPIO16)
- new net M_OE: J11.13 (Pin_13), U2.26 (ADC2_CH0/GPIO4), U7.23 (~{OE})
- new net PCA_A1: JP1.2 (B), R18.2, U7.2 (A1)
- new net PCA_A2: JP2.2 (B), R19.2, U7.3 (A2)
- new net PCA_A3: JP3.2 (B), R20.2, U7.4 (A3)
- new net PCA_A4: JP4.2 (B), R21.2, U7.5 (A4)
- new net PCA_A5: JP5.2 (B), R22.2, U7.24 (A5)
- new net PWR_LED_2: D25.2 (A), R23.2
- new net SBC_VIN_BUCK: C7.1, SW1.2, U8.1 (VIN)
- new net SBC_VSS: C8.1, J16.1 (VBUS), L2.2, R23.1, U8.4 (FB)
- no-connect marks 4 -> 14
Other:
- sheet motor_driver_1 ports: added none; removed MA2_IN, MB2_IN
- sheet motor_driver_2 ports: added none; removed MA2_IN, MB2_IN
- moved on the sheet: C5, C6, D17, D18, D19, D20, D21, D22, D23, H1, H2, H3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

Commit message: done placement again
Parts:
- removed C5, C7: 100uF, Capacitor_THT:C_Radial_D6.3mm_H11.0mm_P2.50mm, symbol Device:C
- removed C6, C8: 1mF, Capacitor_THT:C_Radial_D8.0mm_H11.5mm_P3.50mm, symbol Device:C
- removed D17, D24: 1N5822, Diode_THT:D_DO-201AD_P15.24mm_Horizontal, symbol Diode:1N5822
- removed L1, L2: 100mH, Inductor_SMD:L_6.3x6.3_H3, symbol Device:L
- removed U4, U8: LM2576HVT-5, Package_TO_SOT_THT:TO-220-5_Horizontal_TabDown, symbol Regulator_Switching:LM2576HVT-5
Connections:
- net SBC_VIN_BUCK renamed buck2/VIN
- net SBC_VSS renamed buck2/VOUT
- net VIN_BUCK renamed BUCK_VS
Other:
- added sheet buck1 (buck-converter.kicad_sch)
- added sheet buck2 (buck-converter.kicad_sch)
- moved on the sheet: D22, D25, H1, H2, H3, H4, J16, J9, R23, R9, SW1

Commit message: done!?!?!
Parts:
- added JP0: A0, Jumper:SolderJumper-2_P1.3mm_Open_Pad1.0x1.5mm, symbol Jumper:SolderJumper_2_Open
- added R28: 10k, Resistor_SMD:R_1206_3216Metric_Pad1.30x1.75mm_HandSolder, symbol Device:R
- JP1: value SolderJumper_2_Open -> A1
- JP2: value SolderJumper_2_Open -> A2
- JP3: value SolderJumper_2_Open -> A3
- JP4: value SolderJumper_2_Open -> A4
- JP5: value SolderJumper_2_Open -> A5
Connections:
- net GPIO16 is gone; now on net INT: J11.12 (Pin_12), U2.27 (GPIO16)
- net GPIO23 is gone; now on net FSYNC: J11.2 (Pin_2), U2.37 (GPIO23)
- net +3.3V: now also JP0.1 (A); no longer U7.1 (A0)
- net 1MA1_ENC: now also J11.11 (Pin_11), J13.3 (Pin_3), U2.28 (GPIO17); no longer J11.8 (Pin_8), J12.3 (Pin_3), U2.31 (GPIO19)
- net 1MA2_ENC: now also J11.10 (Pin_10), J13.4 (Pin_4), U2.29 (GPIO5); no longer J11.9 (Pin_9), J12.4 (Pin_4), U2.30 (GPIO18)
- net 1MB1_ENC: now also J10.12 (Pin_12), J15.3 (Pin_3), U2.12 (MTMS/GPIO14/ADC2_CH6); no longer J11.11 (Pin_11), J13.3 (Pin_3), U2.28 (GPIO17)
- net 1MB1_IN: now also U7.10 (LED4); no longer U7.11 (LED5)
- net 1MB2_ENC: now also J10.13 (Pin_13), J15.4 (Pin_4), U2.13 (MTDI/GPIO12/ADC2_CH5); no longer J11.10 (Pin_10), J13.4 (Pin_4), U2.29 (GPIO5)
- net 1MB_EN: now also U7.9 (LED3); no longer U7.10 (LED4)
- net 2MA1_ENC: now also J11.8 (Pin_8), J12.3 (Pin_3), U2.31 (GPIO19); no longer J10.10 (Pin_10), J14.3 (Pin_3), U2.10 (DAC_2/ADC2_CH9/GPIO26)
- net 2MA2_ENC: now also J11.9 (Pin_9), J12.4 (Pin_4), U2.30 (GPIO18); no longer J10.11 (Pin_11), J14.4 (Pin_4), U2.11 (ADC2_CH7/GPIO27)
- net 2MB1_ENC: now also J10.10 (Pin_10), J14.3 (Pin_3), U2.10 (DAC_2/ADC2_CH9/GPIO26); no longer J10.12 (Pin_12), J15.3 (Pin_3), U2.12 (MTMS/GPIO14/ADC2_CH6)
- net 2MB1_IN: now also U7.18 (LED11); no longer U7.17 (LED10)
- net 2MB2_ENC: now also J10.11 (Pin_11), J14.4 (Pin_4), U2.11 (ADC2_CH7/GPIO27); no longer J10.13 (Pin_13), J15.4 (Pin_4), U2.13 (MTDI/GPIO12/ADC2_CH5)
- net 2MB_EN: now also U7.19 (LED12); no longer U7.18 (LED11)
- net FSYNC: no longer J10.7 (Pin_7), U2.7 (32K_XP/GPIO32/ADC1_CH4)
- net GND: now also R28.1
- net INT: no longer J10.8 (Pin_8), U2.8 (32K_XN/GPIO33/ADC1_CH5)
- net 2MB2_IN: now reaches U7.20 (LED13)
- net 1MB2_IN: now reaches U7.8 (LED2)
- new net 1MA2_IN: U7.11 (LED5)
- new net 2MA2_IN: U7.17 (LED10)
- new net GPIO32: J10.7 (Pin_7), U2.7 (32K_XP/GPIO32/ADC1_CH4)
- new net GPIO33: J10.8 (Pin_8), U2.8 (32K_XN/GPIO33/ADC1_CH5)
- new net PCA_A0: JP0.2 (B), R28.2, U7.1 (A0)
- no-connect marks 14 -> 10
Other:
- sheet motor_driver_1 ports: added MA2_IN, MB2_IN; removed none
- sheet motor_driver_2 ports: added MA2_IN, MB2_IN; removed none
- moved on the sheet: D18, D19, D20, D21, D23, H1, H2, H3, H4, J10, J11, J12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
