File: int-brain.kicad_sch (KiCad schematic)
At the start: 62 parts, among them J1 Top, J10 2MB, J11 1MB, J12 1MA, J13 1MA_ENC, J14 1MB_ENC, J15 2MA_ENC, J16 MPU9250, J17 VBATT_SELECT, J2 Bottom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

Commit message: change I2C and minor updates
Parts:
- added J18: I2C0, Connector_JST:JST_EH_B3B-EH-A_1x03_P2.50mm_Vertical, symbol Connector:Conn_01x03_Pin
- added R32, R33: 4.7k, Resistor_SMD:R_1206_3216Metric_Pad1.30x1.75mm_HandSolder, symbol Device:R
- J7: value I2C0 -> I2C1
- JP7: value I/O -> A6
Connections:
- net +3.3V: now also R32.2, R33.2
- net GND: now also J18.1 (Pin_1)
- net SCL0: now also J18.2 (Pin_2); no longer J7.2 (Pin_2)
- net SDA0: now also J18.3 (Pin_3); no longer J7.3 (Pin_3)
- net GPIO13 renamed SDA1
- net SDA1: now also J7.3 (Pin_3), R33.1
- net GPIO15 renamed SCL1
- net SCL1: now also J7.2 (Pin_2), R32.1
- net PCA_IO renamed PCA_A6
Other:
- note added: "A second I2C port is needed to allow the ESP32 to act as a slave to another SBC such as a Raspberry Pi or an NVIDIA Jetson."
- note added: "Protocol pins (I2C0 and UART0) are chosen to keep compliance with the Arduino framework, even though this is unlikely to be used with this board. Most other GPIO are chosen based on physical proximity to peripherals and ease of routing the PCB."
- note removed: "Default I/O to output mode by pull-down."
- note removed: "Protocol pins (I2C and UART0) are chosen to keep compliance with the Arduino framework, even though this is unlikely to be used with this board. Most other GPIO are chosen based on physical proximity to peripherals and ease of routing the PCB."
- moved on the sheet: J1, J13, J14, J15, J2, J6, J7, J8, R15, R16, U2

Commit message: done?
Connections:
- net +3.3V: now also J16.10 (Pin_10)
- net VSS: no longer J16.10 (Pin_10)
Changed lines of the file:
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@@
+	)
+	(symbol
+		(lib_id "power:+3.3V")
+		(at 367.03 459.74 0)
+		(unit 1)
+		(exclude_from_sim no)
+		(in_bom yes)
+		(on_board yes)
+		(dnp no)
+		(fields_autoplaced yes)
+		(property "Reference" "#PWR031"
+			(at 367.03 463.55 0)
+			(effects
+				(font
+					(size 1.27 1.27)
+				)
+				(hide yes)
+			)
+		)
+		(property "Value" "+3.3V"
+			(at 367.03 454.66 0)
+			(effects
+				(font
+					(size 1.27 1.27)
+				)
+			)
+		)
+		(property "Footprint" ""
+			(at 367.03 459.74 0)
+			(effects
+				(font
+					(size 1.27 1.27)
+				)
+				(hide yes)
+			)
+		)
+		(property "Datasheet" ""
+			(at 367.03 459.74 0)
+			(effects
+				(font
+					(size 1.27 1.27)
+				)
+				(hide yes)
+			)
+		)
+		(property "Description" "Power symbol creates a global label with name \"+3.3V\""
+			(at 367.03 459.74 0)
+			(effects
+				(font
+					(size 1.27 1.27)
+				)
+				(hide yes)
+			)
+		)
+		(pin "1"
+		)
+		(instances
+			(project ""
+				(path "/177c6115-ec2a-43b1-88e2-eca3e5dd1279"
+					(reference "#PWR031")
+					(unit 1)
+				)
+			)
+		)
 	)
 	(symbol
@@
 					(unit 1)
 				)
-			)
-		)
-	)
-	(symbol
-		(lib_id "power:VSS")
-		(at 367.03 459.74 0)
-		(unit 1)
-		(exclude_from_sim no)
-		(in_bom yes)
-		(on_board yes)
-		(dnp no)
-		(fields_autoplaced yes)
-		(property "Reference" "#PWR031"
-			(at 367.03 463.55 0)
-			(effects
-				(font
-					(size 1.27 1.27)
-				)
-				(hide yes)
-			)
-		)
-		(property "Value" "VSS"
-			(at 367.03 454.66 0)
-			(effects
-				(font
-					(size 1.27 1.27)
-				)
-			)
-		)
-		(property "Footprint" ""
-			(at 367.03 459.74 0)
-			(effects
-				(font
-					(size 1.27 1.27)
-				)
-				(hide yes)
-			)
-		)
-		(property "Datasheet" ""
-			(at 367.03 459.74 0)
-			(effects
-				(font
-					(size 1.27 1.27)
-				)
-				(hide yes)
-			)
-		)
-		(property "Description" "Power symbol creates a global label with name \"VSS\""
-			(at 367.03 459.74 0)
-			(effects
-				(font
-					(size 1.27 1.27)
-				)
-				(hide yes)
-			)
-		)
-		(pin "1"
-		)
-		(instances
-			(project "int-brain"
-				(path "/177c6115-ec2a-43b1-88e2-eca3e5dd1279"
-					(reference "#PWR031")
-					(unit 1)
-				)

Commit message: finally done?
Parts:
- R14: value 470R -> 220R
Connections:
- net +3.3V: now also R14.1
- net VSS: no longer R14.1
Other:
- moved on the sheet: C26, C27, D7, R14
Changed lines of the file:
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@@
 	)
 	(junction
-		(at 130.81 519.43)
-		(diameter 0)
-		(color 0 0 0 0)
-	)
-	(junction
 		(at 118.11 377.19)
 		(diameter 0)
@@
 	)
 	(junction
-		(at 55.88 535.94)
+		(at 55.88 519.43)
 		(diameter 0)
 		(color 0 0 0 0)
 	)
 	(junction
-		(at 55.88 519.43)
+		(at 325.12 105.41)
 		(diameter 0)
 		(color 0 0 0 0)
 	)
 	(junction
-		(at 325.12 105.41)
+		(at 187.96 476.25)
 		(diameter 0)
 		(color 0 0 0 0)
@@
 	)
 	(junction
+		(at 201.93 459.74)
+		(diameter 0)
+		(color 0 0 0 0)
+	)
+	(junction
 		(at 123.19 494.03)
 		(diameter 0)
@@
 	)
 	(junction
-		(at 157.48 467.36)
+		(at 157.48 476.25)
 		(diameter 0)
 		(color 0 0 0 0)
@@
 	)
 	(junction
-		(at 173.99 467.36)
+		(at 173.99 476.25)
 		(diameter 0)
 		(color 0 0 0 0)
@@
 	(wire
 		(pts
-			(xy 55.88 535.94) (xy 144.78 535.94)
-		)
-		(stroke
-			(width 0)
-			(type default)
-		)
-	)
-	(wire
-		(pts
 			(xy 88.9 369.57) (xy 88.9 393.7)
 		)
@@
 	(wire
 		(pts
+			(xy 157.48 476.25) (xy 157.48 471.17)
+		)
+		(stroke
+			(width 0)
+			(type default)
+		)
+	)
+	(wire
+		(pts
 			(xy 120.65 29.21) (xy 120.65 31.75)
 		)
@@
 	(wire
 		(pts
-			(xy 149.86 471.17) (xy 149.86 467.36)
+			(xy 149.86 480.06) (xy 149.86 476.25)
 		)
 		(stroke
@@
 	(wire
 		(pts
-			(xy 144.78 519.43) (xy 144.78 525.78)
+			(xy 219.71 459.74) (xy 219.71 464.82)
 		)
 		(stroke
@@
 	(wire
 		(pts
-			(xy 144.78 533.4) (xy 144.78 535.94)
+			(xy 187.96 463.55) (xy 187.96 459.74)
+		)
+		(stroke
+			(width 0)
+			(type default)
+		)
+	)
+	(wire
+		(pts
+			(xy 219.71 472.44) (xy 219.71 476.25)
 		)
 		(stroke
@@
 	(wire
 		(pts
-			(xy 173.99 467.36) (xy 187.96 467.36)
+			(xy 173.99 476.25) (xy 187.96 476.25)
 		)
 		(stroke
@@
 	(wire
 		(pts
+			(xy 187.96 476.25) (xy 187.96 471.17)
+		)
+		(stroke
+			(width 0)
+			(type default)
+		)
+	)
+	(wire
+		(pts
 			(xy 236.22 90.17) (xy 384.81 90.17)
 		)
@@
 	(wire
 		(pts
-			(xy 142.24 519.43) (xy 144.78 519.43)
+			(xy 217.17 459.74) (xy 219.71 459.74)
 		)
 		(stroke
@@
 	(wire
 		(pts
+			(xy 173.99 476.25) (xy 173.99 467.36)
+		)
+		(stroke
+			(width 0)
+			(type default)
+		)
+	)
+	(wire
+		(pts
 			(xy 52.07 524.51) (xy 41.91 524.51)
 		)
@@
 	(wire
 		(pts
+			(xy 187.96 476.25) (xy 219.71 476.25)
+		)
+		(stroke
+			(width 0)
+			(type default)
+		)
+	)
+	(wire
+		(pts
 			(xy 236.22 102.87) (xy 384.81 102.87)
 		)
@@
 	(wire
 		(pts
-			(xy 149.86 467.36) (xy 157.48 467.36)
+			(xy 149.86 476.25) (xy 157.48 476.25)
 		)
 		(stroke
@@
 	(wire
 		(pts
+			(xy 201.93 459.74) (xy 209.55 459.74)
+		)
+		(stroke
+			(width 0)
+			(type default)
+		)
+	)
+	(wire
+		(pts
 			(xy 345.44 133.35) (xy 345.44 146.05)
 		)
@@
 	(wire
 		(pts
-			(xy 157.48 467.36) (xy 173.99 467.36)
+			(xy 157.48 476.25) (xy 173.99 476.25)
 		)
 		(stroke
@@
 		)
 	)
+	(wire
+		(pts
+			(xy 157.48 463.55) (xy 157.48 459.74)
+		)
+		(stroke
+			(width 0)
+			(type default)
+		)
+	)
 	(bus
 		(pts
@@
 	(wire
 		(pts
-			(xy 130.81 519.43) (xy 134.62 519.43)
-		)
-		(stroke
-			(width 0)
-			(type default)
-		)
-	)
-	(wire
-		(pts
 			(xy 236.22 77.47) (xy 307.34 77.47)
 		)
@@
 	(text "3.3V LDO"
 		(exclude_from_sim no)
-		(at 176.784 474.472 0)
+		(at 156.21 437.388 0)
 		(effects
 			(font
@@
 	)
 	(label "PWR_LED_1"
-		(at 144.78 519.43 0)
+		(at 219.71 459.74 0)
 		(fields_autoplaced yes)
 		(effects
@@
 	(symbol
 		(lib_id "Device:R")
-		(at 138.43 519.43 90)
+		(at 213.36 459.74 90)
 		(unit 1)
 		(exclude_from_sim no)
@@
 		(fields_autoplaced yes)
 		(property "Reference" "R14"
-			(at 138.43 513.08 90)
+			(at 213.36 453.39 90)
 			(effects
 				(font
@@
 			)
 		)
-		(property "Value" "470R"
-			(at 138.43 515.62 90)
+		(property "Value" "220R"
+			(at 213.36 455.93 90)
 			(effects
 				(font
@@
 		)
 		(property "Footprint" "Resistor_SMD:R_1206_3216Metric_Pad1.30x1.75mm_HandSolder"
-			(at 138.43 521.208 90)
+			(at 213.36 461.518 90)
 			(effects
 				(font
@@
 		)
 		(property "Datasheet" "~"
-			(at 138.43 519.43 0)
+			(at 213.36 459.74 0)
 			(effects
 				(font
@@
 		)
 		(property "Description" "Resistor"
-			(at 138.43 519.43 0)
+			(at 213.36 459.74 0)
 			(effects
 				(font
@@
 	(symbol
 		(lib_id "power:GND")
-		(at 149.86 471.17 0)
+		(at 149.86 480.06 0)
 		(unit 1)
 		(exclude_from_sim no)
@@
 		(fields_autoplaced yes)
 		(property "Reference" "#PWR058"
-			(at 149.86 477.52 0)
+			(at 149.86 486.41 0)
 			(effects
 				(font
@@
 		)
 		(property "Value" "GND"
-			(at 149.86 476.25 0)
+			(at 149.86 485.14 0)
 			(effects
 				(font
@@
 		)
 		(property "Footprint" ""
-			(at 149.86 471.17 0)
+			(at 149.86 480.06 0)
 			(effects
 				(font
@@
 		)
 		(property "Datasheet" ""
-			(at 149.86 471.17 0)
+			(at 149.86 480.06 0)
 			(effects
 				(font
@@
 		)
 		(property "Description" "Power symbol creates a global label with name \"GND\" , ground"
-			(at 149.86 471.17 0)
+			(at 149.86 480.06 0)
 			(effects
 				(font
@@
 	(symbol
 		(lib_id "Device:C")
-		(at 187.96 463.55 0)
+		(at 187.96 467.36 0)
 		(unit 1)
 		(exclude_from_sim no)
@@
 		(fields_autoplaced yes)
 		(property "Reference" "C27"
-			(at 191.77 462.2799 0)
+			(at 191.77 466.0899 0)
 			(effects
 				(font
@@
 		)
 		(property "Value" "10uF"
-			(at 191.77 464.8199 0)
+			(at 191.77 468.6299 0)
 			(effects
 				(font
@@
 		)
 		(property "Footprint" "Capacitor_SMD:C_1206_3216Metric_Pad1.33x1.80mm_HandSolder"
-			(at 188.9252 467.36 0)
+			(at 188.9252 471.17 0)
 			(effects
 				(font
@@
 		)
 		(property "Datasheet" "~"
-			(at 187.96 463.55 0)
+			(at 187.96 467.36 0)
 			(effects
 				(font
@@
 		)
 		(property "Description" "Unpolarized capacitor"
-			(at 187.96 463.55 0)
+			(at 187.96 467.36 0)
 			(effects
 				(font
@@
 	(symbol
 		(lib_id "Device:C")
-		(at 157.48 463.55 0)
+		(at 157.48 467.36 0)
 		(unit 1)
 		(exclude_from_sim no)
@@
 		(fields_autoplaced yes)
 		(property "Reference" "C26"
-			(at 161.29 462.2799 0)
+			(at 161.29 466.0899 0)
 			(effects
 				(font
@@
 		)
 		(property "Value" "10uF"
-			(at 161.29 464.8199 0)
+			(at 161.29 468.6299 0)
 			(effects
 				(font
@@
 		)
 		(property "Footprint" "Capacitor_SMD:C_1206_3216Metric_Pad1.33x1.80mm_HandSolder"
-			(at 158.4452 467.36 0)
+			(at 158.4452 471.17 0)
 			(effects
 				(font
@@
 		)
 		(property "Datasheet" "~"
-			(at 157.48 463.55 0)
+			(at 157.48 467.36 0)
 			(effects
 				(font
@@
 		)
 		(property "Description" "Unpolarized capacitor"
-			(at 157.48 463.55 0)
+			(at 157.48 467.36 0)
 			(effects
 				(font
@@
 	(symbol
 		(lib_id "Device:LED")
-		(at 144.78 529.59 90)
+		(at 219.71 468.63 90)
 		(unit 1)
 		(exclude_from_sim no)
@@
 		(dnp no)
 		(property "Reference" "D7"
-			(at 146.304 526.796 90)
+			(at 221.234 465.836 90)
 			(effects
 				(font
@@
 		)
 		(property "Value" "PWR"
-			(at 146.304 529.336 90)
+			(at 221.234 468.376 90)
 			(effects
 				(font
@@
 		)
 		(property "Footprint" "LED_SMD:LED_1206_3216Metric_Pad1.42x1.75mm_HandSolder"
-			(at 144.78 529.59 0)
+			(at 219.71 468.63 0)
 			(effects
 				(font
@@
 		)
 		(property "Datasheet" "~"
-			(at 144.78 529.59 0)
+			(at 219.71 468.63 0)
 			(effects
 				(font
@@
 		)
 		(property "Description" "Light emitting diode"
-			(at 144.78 529.59 0)
+			(at 219.71 468.63 0)
 			(effects
 				(font

Commit message: something
Parts:
- added C28, C29, C30: 10uF, Capacitor_SMD:C_1206_3216Metric_Pad1.33x1.80mm_HandSolder, symbol Device:C
Connections:
- net +3.3VA: now also C30.2
- net GND: now also C28.2, C29.2, C30.1
- net VSS: now also C29.1
- net buck2/VOUT: now also C28.1
