File: buck-converter.kicad_sch (KiCad schematic)
At the start: 9 parts, among them U4 TPS5430DDA

Commit message: placed?
Parts:
- removed C5: 4.7uF, Capacitor_SMD:C_Elec_5x5.8, symbol Device:C
- removed C8: 220uF, Capacitor_THT:CP_Radial_D6.3mm_P2.50mm, symbol Device:C_Polarized_US
- removed D17: B340, Diode_SMD:D_SMC_Handsoldering, symbol Diode:B340
- removed U4: TPS5430DDA, Package_SO:TI_SO-PowerPAD-8_ThermalVias, symbol Regulator_Switching:TPS5430DDA
- added C11: 330uF, Capacitor_SMD:CP_Elec_8x10.5, symbol Device:C_Polarized
- added C22, C24: 10nF, Capacitor_SMD:C_0603_1608Metric_Pad1.08x0.95mm_HandSolder, symbol Device:C
- added C8: 4.7uF, Capacitor_SMD:CP_Elec_4x5.4, symbol Device:C_Polarized
- added D8: SS54, Diode_SMD:D_SMA_Handsoldering, symbol Device:D_Schottky
- added U7: ~, Package_SO:SOIC-8-1EP_3.9x4.9mm_P1.27mm_EP2.29x3mm_ThermalVias, symbol TPS5450DDA:TPS5450DDA
- R22: renamed from R25; value 3.24k -> 3.16k
- renumbered C7 to C10, C6 to C9, R24 to R21
Connections:
- net BUCK_OUT: now also D8.1 (K), U7.8 (PH)
- net BUCK_VSENSE: now also U7.4 (VSENSE)
- net GND: now also C11.2, C22.2, C24.2, C8.2, D8.2 (A), U7.6 (GND), U7.9 (Pad)
- net VIN: now also C22.1, C8.1, U7.7 (VIN)
- net VOUT: now also C11.1, C24.1
- net at C10.1: now also U7.1 (BOOT)
- no-connect marks 1 -> 3
Other:
- moved on the sheet: C10, C9, L1, R21, R22

Commit message: minor improvements
Parts:
- U7: value ~ -> TPS5450DDA
Other:
- note added: "As per datasheet ENA is floated to enable the switching IC."
- note added: "Bog-standard buck converter circuit, just read the datasheet for component values and justifications. The symbol is custom (available in the /libraries folder of this project), but uses the standard SOIC-8 footprint."
- note added: "Buck Converter (12 V or 24 V to 5V @ 5A)"
- note added: "TPS5450 Datasheet: https://www.ti.com/lit/ds/symlink/tps5450.pdf"
- company: (none) -> Anuj Verma
- title: (none) -> TPS5450 5V 5A Buck Converter
- moved on the sheet: C10, C11, C22, C24, C8, C9, D8, L1, R21, R22, U7

Commit message: footprint updates
Parts:
- C22, C24, C9: footprint Capacitor_SMD:C_0603_1608Metric_Pad1.08x0.95mm_HandSolder -> Capacitor_SMD:C_0805_2012Metric_Pad1.18x1.45mm_HandSolder
Changed lines of the file:
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@@
 			)
 		)
-		(property "Footprint" "Capacitor_SMD:C_0603_1608Metric_Pad1.08x0.95mm_HandSolder"
+		(property "Footprint" "Capacitor_SMD:C_0805_2012Metric_Pad1.18x1.45mm_HandSolder"
 			(at 68.2752 78.74 0)
 			(effects
@@
 			)
 		)
-		(property "Footprint" "Capacitor_SMD:C_0603_1608Metric_Pad1.08x0.95mm_HandSolder"
+		(property "Footprint" "Capacitor_SMD:C_0805_2012Metric_Pad1.18x1.45mm_HandSolder"
 			(at 202.8952 81.28 0)
 			(effects
@@
 			)
 		)
-		(property "Footprint" "Capacitor_SMD:C_0603_1608Metric_Pad1.08x0.95mm_HandSolder"
+		(property "Footprint" "Capacitor_SMD:C_0805_2012Metric_Pad1.18x1.45mm_HandSolder"
 			(at 79.7052 78.74 0)
 			(effects
